Commit message: modify

File: urdf/robots/kobuki_hexagons_asus_xtion_pro.urdf.xacro (robot description, xacro)
@@ -4,5 +4,4 @@
     - Stacks    : hexagons
     - 3d Sensor : asus_xtion_pro
-    - 2d sensor : hokuyo scanner
 -->
 <robot name="turtlebot" xmlns:xacro="http://ros.org/wiki/xacro">
@@ -10,8 +9,8 @@
   <xacro:include filename="$(find kobuki_description)/urdf/kobuki.urdf.xacro" />
   <xacro:include filename="$(find turtlebot_description)/urdf/stacks/hexagons.urdf.xacro"/>
+  <!--
   <xacro:include filename="$(find turtlebot_description)/urdf/sensors/asus_xtion_pro.urdf.xacro"/>
-  <!--
+  -->
   <xacro:include filename="$(find MultiViewSLAM)/urdf/sensors/asus_xtion_pro.urdf.xacro"/>
-  -->
   <!--  <xacro:include filename="$(find MultiViewSLAM)/urdf/sensors/hokuyo.urdf.xacro"/>
     <xacro:sensor_hokuyo name="laser" parent="base_link">
@@ -21,4 +20,4 @@
   <kobuki/>
   <stack_hexagons                 parent="base_link"/>
-  <sensor_asus_xtion_pro          parent="base_link"/>
+  <xacro:sensor_asus_xtion_pro          parent="base_link"/>
 </robot>

File: urdf/sensors/asus_xtion_pro.urdf.xacro (robot description, xacro)
@@ -1,92 +1,94 @@
 <?xml version="1.0"?>
-<robot xmlns:xacro="http://ros.org/wiki/xacro">
-    <xacro:property name="M_PI" value="3.1415926535897931" />
-    <xacro:macro name="asus_camera_model" params="name parent *origin">
-        <joint name="${name}_joint" type="fixed">
-            <xacro:insert_block name="origin" />
-            <parent link="${parent}"/>
-            <child link="${name}_link"/>
-        </joint>
-        <link name="${name}_link">
-            <inertial>
-                <mass value="0.200" />
-                <origin xyz="0 0 0" rpy="0 0 0" />
-                <inertia ixx="5.8083e-4" ixy="0" ixz="0" iyy="3.0833e-5" iyz="0" izz="5.9083e-4" />
-            </inertial>
-            <visual>
-            <origin xyz="0 0 0" rpy="0 0 0" />
-            <geometry>
-                <mesh filename="package://hector_sensors_description/meshes/asus_camera/asus_camera_simple.dae"/>
-            </geometry>
-            </visual>
-            <collision>
-            <origin xyz="0 0 0" rpy="0 0 0" />
-            <geometry>
-                <box size="0.035 0.185 0.025"/>
-            </geometry>
-            </collision>
-        </link>
-        <joint name="${name}_depth_joint" type="fixed">
-            <origin xyz="0.0 0.049 0.0" rpy="0 0 0" />
-            <parent link="${name}_link" />
-            <child link="${name}_depth_frame"/>
-        </joint>
-        <link name="${name}_depth_frame"/>
-        <joint name="${name}_depth_optical_joint" type="fixed">
-            <origin xyz="0 0 0" rpy="${-M_PI/2} 0.0 ${-M_PI/2}" />
-            <parent link="${name}_depth_frame" />
-            <child link="${name}_depth_optical_frame"/>
-        </joint>
-        <link name="${name}_depth_optical_frame"/>
-        <joint name="${name}_rgb_joint" type="fixed">
-            <origin xyz="0.0 0.022 0.0" rpy="0 0 0" />
-            <parent link="${name}_link" />
-            <child link="${name}_rgb_frame"/>
-        </joint>
-        <link name="${name}_rgb_frame"/>
-        <joint name="${name}_rgb_optical_joint" type="fixed">
-            <origin xyz="0 0 0" rpy="${-M_PI/2} 0.0 ${-M_PI/2}" />
-            <parent link="${name}_rgb_frame" />
-            <child link="${name}_rgb_optical_frame"/>
-        </joint>
-        <link name="${name}_rgb_optical_frame"/>
-    </xacro:macro>
-    <xacro:macro name="asus_camera" params="name parent *origin">
-        <xacro:asus_camera_model name="${name}" parent="${parent}">
-            <xacro:insert_block name="origin" />
-        </xacro:asus_camera_model>
-        <!-- ASUS Xtion PRO camera for simulation -->
-        <gazebo reference="${name}_depth_frame">
-            <sensor type="depth" name="${name}">
-                <update_rate>20</update_rate>
-                <camera>
-                    <horizontal_fov>${62.8 * M_PI/180.0}</horizontal_fov>
-                    <image>
-                        <format>R8G8B8</format>
-                        <width>640</width>
-                        <height>480</height>
-                    </image>
-                    <clip>
-                        <near>0.5</near>
-                        <far>9</far>
-                    </clip>
-                </camera>
-                <plugin name="${name}_camera_controller" filename="libgazebo_ros_openni_kinect.so">
-                    <alwaysOn>true</alwaysOn>
-                    <updateRate>20</updateRate>
-                    <imageTopicName>${name}/rgb/image_raw</imageTopicName>
-                    <cameraInfoTopicName>${name}/rgb/camera_info</cameraInfoTopicName>
-                    <depthImageTopicName>${name}/depth/image_raw</depthImageTopicName>
-                    <depthImageCameraInfoTopicName>${name}/depth/camera_info</depthImageCameraInfoTopicName>
-                    <pointCloudTopicName>${name}/depth/points</pointCloudTopicName>
-                    <frameName>${name}_depth_optical_frame</frameName>
-                    <distortion_k1>0.0</distortion_k1>
-                    <distortion_k2>0.0</distortion_k2>
-                    <distortion_k3>0.0</distortion_k3>
-                    <distortion_t1>0.0</distortion_t1>
-                    <distortion_t2>0.0</distortion_t2>
-                </plugin>
-            </sensor>
-        </gazebo>
-    </xacro:macro>
+<robot name="sensor_asus_xtion_pro" xmlns:xacro="http://ros.org/wiki/xacro">
+  <xacro:include filename="$(find turtlebot_description)/urdf/turtlebot_gazebo.urdf.xacro"/>
+  <xacro:include filename="$(find turtlebot_description)/urdf/turtlebot_properties.urdf.xacro"/>
+  <!-- Xacro properties -->
+  <xacro:property name="M_SCALE" value="0.001"/>
+  <xacro:property name="asus_xtion_pro_cam_py" value="0.0205"/>
+  <xacro:property name="asus_xtion_pro_depth_rel_rgb_py" value="0.0270" />
+  <xacro:property name="asus_xtion_pro_cam_rel_rgb_py"   value="-0.0220" />
+  <!-- Parameterised in part by the values in turtlebot_properties.urdf.xacro -->
+  <xacro:macro name="sensor_asus_xtion_pro" params="parent">
+    <joint name="camera_rgb_joint" type="fixed">
+      <origin xyz="${cam_px} ${asus_xtion_pro_cam_py} ${cam_pz}"
+              rpy="${cam_or} ${cam_op} ${cam_oy}"/>
+      <parent link="${parent}"/>
+      <child link="camera_rgb_frame" />
+    </joint>
+    <link name="camera_rgb_frame"/>
+    <joint name="camera_rgb_optical_joint" type="fixed">
+      <origin xyz="0 0 0" rpy="${-M_PI/2} 0 ${-M_PI/2}" />
+      <parent link="camera_rgb_frame" />
+      <child link="camera_rgb_optical_frame" />
+    </joint>
+    <link name="camera_rgb_optical_frame"/>
+    <joint name="camera_joint" type="fixed">
+      <origin xyz="0 ${asus_xtion_pro_cam_rel_rgb_py} 0"
+              rpy="0 0 0"/>
+      <parent link="camera_rgb_frame"/>
+      <child link="camera_link"/>
+    </joint>
+    <link name="camera_link">
+      <visual>
+        <origin xyz="-0.015 0.0035 0.004" rpy="0 0 0"/>
+        <geometry>
+          <mesh filename="package://turtlebot_description/meshes/sensors/xtion_pro_camera.dae"/>
+        </geometry>
+      </visual>
+      <collision>
+        <origin xyz="0.0 0.0 0.0" rpy="0 0 0" />
+        <geometry>
+        <box size="0.0730 0.2760 0.0720"/>
+      </geometry>
+      </collision>
+      <inertial>
+        <mass value="0.170" />
+        <origin xyz="0 0 0" />
+        <inertia ixx="0.001152600" ixy="0.0" ixz="0.0"
+                 iyy="0.000148934" iyz="0.0"
+                 izz="0.001154654" />
+      </inertial>
+    </link>
+    <joint name="camera_depth_joint" type="fixed">
+      <origin xyz="0 ${asus_xtion_pro_depth_rel_rgb_py} 0" rpy="0 0 0" />
+      <parent link="camera_rgb_frame" />
+      <child link="camera_depth_frame" />
+    </joint>
+    <link name="camera_depth_frame"/>
+    <joint name="camera_depth_optical_joint" type="fixed">
+      <origin xyz="0 0 0" rpy="${-M_PI/2} 0 ${-M_PI/2}" />
+      <parent link="camera_depth_frame" />
+      <child link="camera_depth_optical_frame" />
+    </joint>
+    <link name="camera_depth_optical_frame"/>
+    <!-- RGBD sensor for simulation, same as Kinect -->
+    <turtlebot_sim_3dsensor/>
+    <!-- Asus mount -->
+    <joint name="mount_asus_xtion_pro_joint" type="fixed">
+      <origin xyz="-0.1024 0.0 0.272" rpy="0 0 0"/>
+      <parent link="${parent}"/>
+      <child link="mount_asus_xtion_pro_link"/>
+    </joint>
+    <link name="mount_asus_xtion_pro_link">
+      <visual>
+        <origin xyz="0 0 0" rpy="${-M_PI/2} 0 0"/>
+        <geometry>
+          <mesh filename="package://turtlebot_description/meshes/sensors/xtion_pro_stack.dae"/>
+        </geometry>
+      </visual>
+      <collision>
+        <origin xyz="0.0 0.0 0.0" rpy="0 0 0" />
+        <geometry>
+        <box size="0.0330 0.2760 0.0120"/>
+      </geometry>
+      </collision>
+      <inertial>
+        <mass value="0.170" />
+        <origin xyz="0 0 0" />
+        <inertia ixx="0.001152600" ixy="0.0" ixz="0.0"
+                 iyy="0.000148934" iyz="0.0"
+                 izz="0.001154654" />
+      </inertial>
+    </link>
+  </xacro:macro>
 </robot>
